Commit message: k

File: description/gazebo_control.xacro (robot description, xacro)
@@ -15,12 +15,12 @@
             <publish_wheel_tf>true</publish_wheel_tf>
         </plugin>
-        <plugin name="gazebo_ros_joint_state_publisher"
+        <!--plugin name="gazebo_ros_joint_state_publisher"
             filename="libgazebo_ros_joint_state_publisher.so">
             <update_rate>20</update_rate>
-            <joint_name>chassis_joint</joint_name>
+            <joint_name>chassis_bottom_joint</joint_name>
             <joint_name>right_wheel_joint</joint_name>
             <joint_name>left_wheel_joint</joint_name>
             <joint_name>caster_weel_joint</joint_name>
-        </plugin>
+        </plugin> -->
     </gazebo>
 </robot>

File: description/lidar.xacro (robot description, xacro)
@@ -2,5 +2,5 @@
 <robot xmlns:xacro="http://www.ros.org/wiki/xacro" >
     <joint name="laser_joint" type="fixed">
-        <parent link="chassis"/>
+        <parent link="chassis_mid"/>
         <child link="laser_frame"/>
         <origin xyz="0.1 0 0.175" rpy="0 0 0"/>

File: description/robot_core.xacro (robot description, xacro)
@@ -1,7 +1,22 @@
 <?xml version="1.0"?>
-<robot xmlns:xacro="http://www.ros.org/wiki/xacro"  >
+<robot xmlns:xacro="http://www.ros.org/wiki/xacro" >
     <xacro:include filename="inertial_macros.xacro"/>
+    <xacro:property name="chassis_length" value="0.26586"/>
+    <xacro:property name="chassis_width" value="0.14"/>
+    <xacro:property name="chassis_height" value="0.15"/>
+    <xacro:property name="chassis_mass" value="1.0"/>
+    <xacro:property name="wheel_radius" value="0.04"/>
+    <xacro:property name="wheel_thickness" value="0.0293"/>
+    <xacro:property name="wheel_mass" value="0.2"/>
+    <xacro:property name="wheel_offset_x" value="0.05065"/>
+    <xacro:property name="wheel_offset_y" value="0.08715"/>
+    <xacro:property name="wheel_offset_z" value="0.02725"/>
+    <xacro:property name="caster_wheel_radius" value="0.0205"/>
+    <xacro:property name="caster_wheel_mass" value="0.1"/>
+    <xacro:property name="tussenstuk_length" value="0.0055"/>
+    <xacro:property name="tussenstuk_width" value="0.0055"/>
+    <xacro:property name="tussenstuk_height" value="0.0715"/>
     <material name="white">
-        <color rgba="1 1 1 1"/>
+        <color rgba="1 1 1 1" />
     </material>
     <material name="orange">
@@ -14,42 +29,228 @@
         <color rgba="0 0 0 1"/>
     </material>
-    <material name="red">
-        <color rgba="1 0 0 1"/>
-    </material>
-    <!-- base link-->
+    <!-- BASE LINK -->
     <link name="base_link">
     </link>
-    <!-- bchassislink-->
-    <joint name="chassis_joint" type="fixed">
-        <parent link="base_link"/>
-        <child link="chassis"/>
-        <origin xyz="-0.1 0 0"/>
-    </joint>
-    <link name="chassis">
-        <visual>
-            <origin xyz="0.15 0 0.075" rpy="0 0 0"/>
-            <geometry>
-                <box size="0.3 0.3 0.15"/>
-            </geometry>
-            <material name="white"/>
-        </visual>
-        <collision>
-            <origin xyz="0.15 0 0.075" rpy="0 0 0"/>
-            <geometry>
-                <box size="0.3 0.3 0.15"/>
-            </geometry>
-        </collision>
-        <xacro:inertial_box mass="0.5" x="0.3" y="0.3" z="0.15">
-            <origin xyz="0.15 0 0.075" rpy="0 0 0"/>
-        </xacro:inertial_box>
-    </link>
-    <gazebo reference="chassis">
-        <material>Gazebo/White</material>
-    </gazebo>
-    <!-- leftwheellink-->
+    <!-- CHASSIS BOTTOM LINK -->
+    <joint name="chassis_bottom_joint" type="fixed">
+        <parent link="base_link"/>
+        <child link="chassis_bottom"/>
+        <origin xyz="0 0 0"/>
+    </joint>
+    <link name="chassis_bottom">
+        <visual>
+            <origin xyz="0.09435 0 0" rpy="0 0 ${pi}"/>
+            <geometry>
+                <mesh filename="file://$(find my_bot)/meshes/Onderstel.stl" scale="0.001 0.001 0.001"/>
+            </geometry>
+            <material name="orange"/>
+        </visual>
+        <collision>
+            <origin xyz="0.09435 0 0" rpy="0 0 ${pi}"/>
+            <geometry>
+                <mesh filename="file://$(find my_bot)/meshes/Onderstel.stl" scale="0.001 0.001 0.001"/>
+            </geometry>
+        </collision>
+        <xacro:inertial_box mass="0.072" x="${chassis_length}" y="${chassis_width}" z="${chassis_height}">
+            <origin xyz="${chassis_length/2} 0 ${chassis_height/2}" rpy="0 0 0"/>
+        </xacro:inertial_box>
+    </link>
+    <gazebo reference="chassis_bottom">
+        <material>Gazebo/Wood</material>
+    </gazebo>
+    <!-- LEFT MOTOR BEUGEL LINK  -->
+    <joint name="chassis_beugel_left_link" type="fixed">
+        <parent link="base_link"/>
+        <child link="chassis_beugel_left"/>
+        <origin xyz="-0.013 -0.06875 0" rpy="1.57079632679 0.0 0.0"/>
+    </joint>
+    <link name="chassis_beugel_left">
+        <visual>
+            <origin xyz="0 0 0"/>
+            <geometry>
+                <mesh filename="file://$(find my_bot)/meshes/MotorBeugel.stl" scale="0.001 0.001 0.001"/>
+            </geometry>
+            <material name="black"/>
+        </visual>
+        <collision>
+            <origin xyz="0 0 0"/>
+            <geometry>
+                <mesh filename="file://$(find my_bot)/meshes/MotorBeugel.stl" scale="0.001 0.001 0.001"/>
+            </geometry>
+        </collision>
+        <xacro:inertial_box mass="0.053" x="0.200" y="0.0041" z="0.140">
+            <origin xyz="0.100 0 0.070" rpy="0 0 0"/>
+        </xacro:inertial_box>
+    </link>
+    <gazebo reference="chassis_beugel_left">
+        <material>Gazebo/FlatBlack</material>
+    </gazebo>
+    <!-- RIGHT MOTOR BEUGEL LINK -->
+    <joint name="chassis_beugel_right_link" type="fixed">
+        <parent link="base_link"/>
+        <child link="chassis_beugel_right"/>
+        <origin xyz="0.013 0.06875 0" rpy="1.57079632679 0 3.14159265359"/>
+    </joint>
+    <link name="chassis_beugel_right">
+        <visual>
+            <origin xyz="0 0 0"/>
+            <geometry>
+                <mesh filename="file://$(find my_bot)/meshes/MotorBeugel.stl" scale="0.001 0.001 0.001"/>
+            </geometry>
+            <material name="black"/>
+        </visual>
+        <collision>
+            <origin xyz="0 0 0"/>
+            <geometry>
+                <mesh filename="file://$(find my_bot)/meshes/MotorBeugel.stl" scale="0.001 0.001 0.001"/>
+            </geometry>
+        </collision>
+        <xacro:inertial_box mass="0.053" x="0.200" y="0.0041" z="0.140">
+            <origin xyz="0.100 0 0.070" rpy="0 0 0"/>
+        </xacro:inertial_box>
+    </link>
+    <gazebo reference="chassis_beugel_right">
+        <material>Gazebo/FlatBlack</material>
+    </gazebo>
+    <!-- CHASSIS TUSSEN LINK 1 -->
+    <joint name="chassis_tussen_one_joint" type="fixed">
+        <parent link="base_link"/>
+        <child link="chassis_tussen_one"/>
+        <origin xyz="-0.03565 0.055 -0.006"/>
+    </joint>
+    <link name="chassis_tussen_one">
+        <visual>
+            <origin xyz="0 0 0"/>
+            <geometry>
+                <mesh filename="file://$(find my_bot)/meshes/Tussenstuk.stl" scale="0.001 0.001 0.001"/>
+            </geometry>
+            <material name="black"/>
+        </visual>
+        <collision>
+            <origin xyz="0 0 0"/>
+            <geometry>
+                <mesh filename="file://$(find my_bot)/meshes/Tussenstuk.stl" scale="0.001 0.001 0.001"/>
+            </geometry>
+        </collision>
+        <xacro:inertial_box mass="0.004" x="${tussenstuk_length}" y="${tussenstuk_width}" z="${tussenstuk_height}">
+            <origin xyz="${tussenstuk_length/2} 0 ${tussenstuk_height/2}" rpy="0 0 0"/>
+        </xacro:inertial_box>
+    </link>
+    <gazebo reference="chassis_tussen_one">
+        <material>Gazebo/Grey</material>
+    </gazebo>
+    <!-- CHASSIS TUSSEN LINK 2 -->
+    <joint name="chassis_tussen_two_joint" type="fixed">
+        <parent link="base_link"/>
+        <child link="chassis_tussen_two"/>
+        <origin xyz="-0.03565 -0.055 -0.006"/>
+    </joint>
+    <link name="chassis_tussen_two">
+        <visual>
+            <origin xyz="0 0 0"/>
+            <geometry>
+                <mesh filename="file://$(find my_bot)/meshes/Tussenstuk.stl" scale="0.001 0.001 0.001"/>
+            </geometry>
+            <material name="black"/>
+        </visual>
+        <collision>
+            <origin xyz="0 0 0"/>
+            <geometry>
+                <mesh filename="file://$(find my_bot)/meshes/Tussenstuk.stl" scale="0.001 0.001 0.001"/>
+            </geometry>
+        </collision>
+        <xacro:inertial_box mass="0.004" x="${tussenstuk_length}" y="${tussenstuk_width}" z="${tussenstuk_height}">
+            <origin xyz="${tussenstuk_length/2} 0 ${tussenstuk_height/2}" rpy="0 0 0"/>
+        </xacro:inertial_box>
+    </link>
+    <gazebo reference="chassis_tussen_two">
+        <material>Gazebo/Grey</material>
+    </gazebo>
+    <!-- CHASSIS TUSSEN LINK 3 -->
+    <joint name="chassis_tussen_three_joint" type="fixed">
+        <parent link="base_link"/>
+        <child link="chassis_tussen_three"/>
+        <origin xyz="0.13935 0.060 -0.006"/>
+    </joint>
+    <link name="chassis_tussen_three">
+        <visual>
+            <origin xyz="0 0 0"/>
+            <geometry>
+                <mesh filename="file://$(find my_bot)/meshes/Tussenstuk.stl" scale="0.001 0.001 0.001"/>
+            </geometry>
+            <material name="black"/>
+        </visual>
+        <collision>
+            <origin xyz="0 0 0"/>
+            <geometry>
+                <mesh filename="file://$(find my_bot)/meshes/Tussenstuk.stl" scale="0.001 0.001 0.001"/>
+            </geometry>
+        </collision>
+        <xacro:inertial_box mass="0.004" x="${tussenstuk_length}" y="${tussenstuk_width}" z="${tussenstuk_height}">
+            <origin xyz="${tussenstuk_length/2} 0 ${tussenstuk_height/2}" rpy="0 0 0"/>
+        </xacro:inertial_box>
+    </link>
+    <gazebo reference="chassis_tussen_three">
+        <material>Gazebo/Grey</material>
+    </gazebo>
+    <!-- CHASSIS TUSSEN LINK 4 -->
+    <joint name="chassis_tussen_four_joint" type="fixed">
+        <parent link="base_link"/>
+        <child link="chassis_tussen_four"/>
+        <origin xyz="0.13935 -0.060 -0.006"/>
+    </joint>
+    <link name="chassis_tussen_four">
+        <visual>
+            <origin xyz="0 0 0"/>
+            <geometry>
+                <mesh filename="file://$(find my_bot)/meshes/Tussenstuk.stl" scale="0.001 0.001 0.001"/>
+            </geometry>
+            <material name="black"/>
+        </visual>
+        <collision>
+            <origin xyz="0 0 0"/>
+            <geometry>
+                <mesh filename="file://$(find my_bot)/meshes/Tussenstuk.stl" scale="0.001 0.001 0.001"/>
+            </geometry>
+        </collision>
+        <xacro:inertial_box mass="0.004" x="${tussenstuk_length}" y="${tussenstuk_width}" z="${tussenstuk_height}">
+            <origin xyz="${tussenstuk_length/2} 0 ${tussenstuk_height/2}" rpy="0 0 0"/>
+        </xacro:inertial_box>
+    </link>
+    <gazebo reference="chassis_tussen_four">
+        <material>Gazebo/Grey</material>
+    </gazebo>
+    <!-- CHASSIS MID LINK -->
+    <joint name="chassis_mid_joint" type="fixed">
+        <parent link="base_link"/>
+        <child link="chassis_mid"/>
+        <origin xyz="0.04935 0 0.0541" rpy="0 0 ${pi}"/>
+    </joint>
+    <link name="chassis_mid">
+        <visual>
+            <origin xyz="0 0 0"/>
+            <geometry>
+                <mesh filename="file://$(find my_bot)/meshes/Mid.stl" scale="0.001 0.001 0.001"/>
+            </geometry>
+            <material name="orange"/>
+        </visual>
+        <collision>
+            <origin xyz="0 0 0"/>
+            <geometry>
+                <mesh filename="file://$(find my_bot)/meshes/Mid.stl" scale="0.001 0.001 0.001"/>
+            </geometry>
+        </collision>
+        <xacro:inertial_box mass="0.053" x="0.200" y="0.0041" z="0.140">
+            <origin xyz="0.100 0 0.070" rpy="0 0 0"/>
+        </xacro:inertial_box>
+    </link>
+    <gazebo reference="chassis_mid">
+        <material>Gazebo/Wood</material>
+    </gazebo>
+    <!-- LEFT WHEEL LINK -->
     <joint name="left_wheel_joint" type="continuous">
-        <parent link="base_link"/>
+        <parent link="chassis_beugel_left"/>
         <child link="left_wheel"/>
-        <origin xyz="0 0.175 0" rpy="-${pi/2} 0 0"/>
+        <origin xyz="0.013 0.02 0.026" rpy="0 ${pi} 0" />
         <axis xyz="0 0 1"/>
     </joint>
@@ -57,5 +258,5 @@
         <visual>
             <geometry>
-                <cylinder radius="0.05" length="0.04"/>
+                <cylinder radius="${wheel_radius}" length="${wheel_thickness}"/>
             </geometry>
             <material name="blue"/>
@@ -63,25 +264,25 @@
         <collision>
             <geometry>
-                <cylinder radius="0.05" length="0.04"/>
-            </geometry>
-        </collision>
-        <xacro:inertial_cylinder mass="0.1" length="0.04" radius="0.05">
+                <sphere radius="${wheel_radius}"/>
+            </geometry>
+        </collision>
+        <xacro:inertial_cylinder mass="${wheel_mass}" length="${wheel_thickness}" radius="${wheel_radius}">
             <origin xyz="0 0 0" rpy="0 0 0"/>
         </xacro:inertial_cylinder>
     </link>
     <gazebo reference="left_wheel">
-        <material>Gazebo/Blue</material>
-    </gazebo>
-    <!--rightwheel-->
+        <material>Gazebo/RedBright</material>
+    </gazebo>
+    <!-- RIGHT WHEEL LINK -->
     <joint name="right_wheel_joint" type="continuous">
-            <parent link="base_link"/>
-            <child link="right_wheel"/>
-            <origin xyz="0 -0.175 0" rpy="${pi/2} 0 0"/>
-            <axis xyz="0 0 -1"/>
+        <parent link="chassis_beugel_right"/>
+        <child link="right_wheel"/>
+        <origin xyz="0.013 0.02 0.026" rpy="0 0 0" />
+        <axis xyz="0 0 1"/>
     </joint>
     <link name="right_wheel">
         <visual>
             <geometry>
-                <cylinder radius="0.05" length="0.04"/>
+                <cylinder radius="${wheel_radius}" length="${wheel_thickness}"/>
             </geometry>
             <material name="blue"/>
@@ -89,38 +290,38 @@
         <collision>
             <geometry>
-                <cylinder radius="0.05" length="0.04"/>
-            </geometry>
-        </collision>
-        <xacro:inertial_cylinder mass="0.1" length="0.04" radius="0.05">
+                <sphere radius="${wheel_radius}"/>
+            </geometry>
+        </collision>
+        <xacro:inertial_cylinder mass="${wheel_mass}" length="${wheel_thickness}" radius="${wheel_radius}">
             <origin xyz="0 0 0" rpy="0 0 0"/>
         </xacro:inertial_cylinder>
     </link>
     <gazebo reference="right_wheel">
-        <material>Gazebo/Blue</material>
-    </gazebo>
-    <!-- casterwiel-->
+        <material>Gazebo/RedBright</material>
+    </gazebo>
+    <!-- CASTER WHEEL LINK -->
     <joint name="caster_wheel_joint" type="fixed">
-        <parent link="chassis"/>
+        <parent link="chassis_bottom"/>
         <child link="caster_wheel"/>
-        <origin xyz="0.24 0 0"/>
+        <origin xyz="0.16935 0 -0.0041" rpy="0 0 1.57079632679"/>
     </joint>
     <link name="caster_wheel">
         <visual>
             <geometry>
-                <sphere radius="0.05"/>
-            </geometry>
-            <material name="black"/>
-        </visual>
-        <collision>
-            <geometry>
-                <sphere radius="0.05"/>
-            </geometry>
-        </collision>
-        <xacro:inertial_sphere mass="0.1" radius="0.05">
+                <mesh filename="file://$(find my_bot)/meshes/CASTER_WIEL.stl" scale="0.001 0.001 0.001"/>
+            </geometry>
+            <material name="white"/>
+        </visual>
+        <collision>
+            <geometry>
+                <mesh filename="file://$(find my_bot)/meshes/CASTER_WIEL.stl" scale="0.001 0.001 0.001"/>
+            </geometry>
+        </collision>
+        <xacro:inertial_sphere mass="${caster_wheel_mass}" radius="${caster_wheel_radius}">
             <origin xyz="0 0 0" rpy="0 0 0"/>
         </xacro:inertial_sphere>
     </link>
     <gazebo reference="caster_wheel">
-        <material>Gazebo/Black</material>
+        <material>Gazebo/White</material>
         <mu1 value="0.001"/>
         <mu2 value="0.001"/>
