Commit message: x

File: description/gazebo_control.xacro (robot description, xacro)
@@ -5,6 +5,6 @@
             <left_joint>left_wheel_joint</left_joint>
             <right_joint>right_wheel_joint</right_joint>
-            <wheel_separation>0.35</wheel_separation>
-            <wheel_diameter>0.1</wheel_diameter>
+            <wheel_separation>0.17430</wheel_separation>
+            <wheel_diameter>0.04</wheel_diameter>
             <max_wheel_torque>200</max_wheel_torque>
             <max_wheel_acceleration>10.0</max_wheel_acceleration>
@@ -15,12 +15,12 @@
             <publish_wheel_tf>true</publish_wheel_tf>
         </plugin>
-        <!--plugin name="gazebo_ros_joint_state_publisher"
+        <plugin name="gazebo_ros_joint_state_publisher"
             filename="libgazebo_ros_joint_state_publisher.so">
             <update_rate>20</update_rate>
-            <joint_name>chassis_bottom_joint</joint_name>
+            <joint_name>chassis_mid_joint</joint_name>
             <joint_name>right_wheel_joint</joint_name>
             <joint_name>left_wheel_joint</joint_name>
             <joint_name>caster_weel_joint</joint_name>
-        </plugin> -->
+        </plugin>
     </gazebo>
 </robot>

File: description/lidar.xacro (robot description, xacro)
@@ -2,7 +2,7 @@
 <robot xmlns:xacro="http://www.ros.org/wiki/xacro" >
     <joint name="laser_joint" type="fixed">
-        <parent link="chassis_mid"/>
+        <parent link="chassis"/>
         <child link="laser_frame"/>
-        <origin xyz="0.1 0 0.175" rpy="0 0 0"/>
+        <origin xyz="0 0 0.5" rpy="0 0 0"/>
     </joint>
     <link name="laser_frame">

File: description/robot.urdf.xacro (robot description, xacro)
@@ -2,5 +2,5 @@
 <robot xmlns:xacro="http://www.ros.org/wiki/xacro"  name="robot">
     <xacro:arg name="use_ros2_control" default="true"/>
-    <xacro:arg name="sim_mode" default="false"/>
+    <xacro:arg name="sim_mode" default="true"/>
     <xacro:if value="$(arg use_ros2_control)">
         <xacro:include filename="ros2_control.xacro" />
@@ -10,4 +10,4 @@
     </xacro:unless>
     <xacro:include filename="robot_core.xacro" />
-    <xacro:include filename="lidar.xacro"/>
+    <!--xacro:include filename="lidar.xacro"/>-->
 </robot>

File: description/robot_core.xacro (robot description, xacro)
@@ -49,5 +49,5 @@
             <origin xyz="0.09435 0 0" rpy="0 0 ${pi}"/>
             <geometry>
-                <mesh filename="file://$(find my_bot)/meshes/Onderstel.stl" scale="0.001 0.001 0.001"/>
+                <box size="0.3 0.14 0.01"/>
             </geometry>
         </collision>
@@ -121,14 +121,14 @@
     <link name="chassis_tussen_one">
         <visual>
-            <origin xyz="0 0 0"/>
-            <geometry>
-                <mesh filename="file://$(find my_bot)/meshes/Tussenstuk.stl" scale="0.001 0.001 0.001"/>
-            </geometry>
-            <material name="black"/>
-        </visual>
-        <collision>
-            <origin xyz="0 0 0"/>
-            <geometry>
-                <mesh filename="file://$(find my_bot)/meshes/Tussenstuk.stl" scale="0.001 0.001 0.001"/>
+            <origin xyz="0 0 0.025"/>
+            <geometry>
+                <cylinder radius="0.01" length= "0.05"/>
+            </geometry>
+            <material name="black"/>
+        </visual>
+        <collision>
+            <origin xyz="0 0 0.025"/>
+            <geometry>
+                <cylinder radius="0.01" length= "0.05"/>
             </geometry>
         </collision>
@@ -148,7 +148,7 @@
     <link name="chassis_tussen_two">
         <visual>
-            <origin xyz="0 0 0"/>
-            <geometry>
-                <mesh filename="file://$(find my_bot)/meshes/Tussenstuk.stl" scale="0.001 0.001 0.001"/>
+            <origin xyz="0 0 0.025"/>
+            <geometry>
+                <cylinder radius="0.01" length= "0.05"/>
             </geometry>
             <material name="black"/>
@@ -175,14 +175,14 @@
     <link name="chassis_tussen_three">
         <visual>
-            <origin xyz="0 0 0"/>
-            <geometry>
-                <mesh filename="file://$(find my_bot)/meshes/Tussenstuk.stl" scale="0.001 0.001 0.001"/>
-            </geometry>
-            <material name="black"/>
-        </visual>
-        <collision>
-            <origin xyz="0 0 0"/>
-            <geometry>
-                <mesh filename="file://$(find my_bot)/meshes/Tussenstuk.stl" scale="0.001 0.001 0.001"/>
+            <origin xyz="0 0 0.025"/>
+            <geometry>
+                <cylinder radius="0.01" length= "0.05"/>
+            </geometry>
+            <material name="black"/>
+        </visual>
+        <collision>
+            <origin xyz="0 0 0.025"/>
+            <geometry>
+                <cylinder radius="0.01" length= "0.05"/>
             </geometry>
         </collision>
@@ -202,14 +202,14 @@
     <link name="chassis_tussen_four">
         <visual>
-            <origin xyz="0 0 0"/>
-            <geometry>
-                <mesh filename="file://$(find my_bot)/meshes/Tussenstuk.stl" scale="0.001 0.001 0.001"/>
-            </geometry>
-            <material name="black"/>
-        </visual>
-        <collision>
-            <origin xyz="0 0 0"/>
-            <geometry>
-                <mesh filename="file://$(find my_bot)/meshes/Tussenstuk.stl" scale="0.001 0.001 0.001"/>
+            <origin xyz="0 0 0.025"/>
+            <geometry>
+                <cylinder radius="0.01" length= "0.05"/>
+            </geometry>
+            <material name="black"/>
+        </visual>
+        <collision>
+            <origin xyz="0 0 0.025"/>
+            <geometry>
+                <cylinder radius="0.01" length= "0.05"/>
             </geometry>
         </collision>
@@ -238,5 +238,5 @@
             <origin xyz="0 0 0"/>
             <geometry>
-                <mesh filename="file://$(find my_bot)/meshes/Mid.stl" scale="0.001 0.001 0.001"/>
+                <box size="0.3 0.14 0.01"/>
             </geometry>
         </collision>
@@ -249,5 +249,5 @@
     </gazebo>
     <!-- LEFT WHEEL LINK -->
-    <joint name="left_wheel_joint" type="continuous">
+    <joint name="right_wheel_joint" type="continuous">
         <parent link="chassis_beugel_left"/>
         <child link="left_wheel"/>
@@ -255,5 +255,5 @@
         <axis xyz="0 0 1"/>
     </joint>
-    <link name="left_wheel">
+    <link name="right_wheel">
         <visual>
             <geometry>
@@ -271,9 +271,9 @@
         </xacro:inertial_cylinder>
     </link>
-    <gazebo reference="left_wheel">
+    <gazebo reference="right_wheel">
         <material>Gazebo/RedBright</material>
     </gazebo>
     <!-- RIGHT WHEEL LINK -->
-    <joint name="right_wheel_joint" type="continuous">
+    <joint name="left_wheel_joint" type="continuous">
         <parent link="chassis_beugel_right"/>
         <child link="right_wheel"/>
@@ -281,5 +281,5 @@
         <axis xyz="0 0 1"/>
     </joint>
-    <link name="right_wheel">
+    <link name="left_wheel">
         <visual>
             <geometry>
@@ -297,5 +297,5 @@
         </xacro:inertial_cylinder>
     </link>
-    <gazebo reference="right_wheel">
+    <gazebo reference="left_wheel">
         <material>Gazebo/RedBright</material>
     </gazebo>
@@ -309,5 +309,5 @@
         <visual>
             <geometry>
-                <mesh filename="file://$(find my_bot)/meshes/CASTER_WIEL.stl" scale="0.001 0.001 0.001"/>
+                <sphere radius="0.015"/>
             </geometry>
             <material name="white"/>
@@ -315,5 +315,5 @@
         <collision>
             <geometry>
-                <mesh filename="file://$(find my_bot)/meshes/CASTER_WIEL.stl" scale="0.001 0.001 0.001"/>
+                <sphere radius="0.015"/>
             </geometry>
         </collision>
@@ -327,3 +327,52 @@
         <mu2 value="0.001"/>
     </gazebo>
+    <joint name="laser_joint" type="fixed">
+        <parent link="chassis_bottom"/>
+        <child link="laser_frame"/>
+        <origin xyz="0.05 0 0.07" rpy="0 0 0"/>
+    </joint>
+    <link name="laser_frame">
+        <visual>
+            <geometry>
+                <cylinder radius="0.05" length="0.04"/>
+            </geometry>
+            <material name="blue"/>
+        </visual>
+        <collision>
+            <geometry>
+                <cylinder radius="0.05" length="0.04"/>
+            </geometry>
+        </collision>
+        <xacro:inertial_cylinder mass="0.1" length="0.04" radius="0.05">
+            <origin xyz="0 0 0" rpy="0 0 0"/>
+        </xacro:inertial_cylinder>
+    </link>
+    <gazebo reference="laser_frame">
+        <material>Gazebo/Blue</material>
+        <sensor name="laser" type="ray">
+            <pose> 0 0 0 0 0 0 </pose>
+            <visualize>true</visualize>
+            <update_rate>10</update_rate>
+            <ray>
+                <scan>
+                    <horizontal>
+                        <samples>360</samples>
+                        <min_angle>-3.14</min_angle>
+                        <max_angle>3.14</max_angle>
+                    </horizontal>
+                </scan>
+                <range>
+                    <min>0.3</min>
+                    <max>12</max>
+                </range>
+            </ray>
+            <plugin name="laser_controller" filename="libgazebo_ros_ray_sensor.so">
+                <ros>
+                    <remapping>~/out:=scan</remapping>
+                </ros>
+                <output_type>sensor_msgs/LaserScan</output_type>
+                <frame_name>laser_frame</frame_name>
+            </plugin>
+        </sensor>
+    </gazebo>
 </robot>
