Commit message: hhah

File: description/robot_core.xacro (robot description, xacro)
@@ -32,4 +32,12 @@
     <link name="base_link">
     </link>
+    <!-- footprint LINK -->
+    <joint name="base_footprint_joint" type="fixed">
+        <parent link="base_link"/>
+        <child link="base_footprint"/>
+        <origin xyz="0 0 0" rpy="0 0 0"/>
+    </joint>
+    <link name="base_footprint">
+    </link>
     <!-- CHASSIS BOTTOM LINK -->
     <joint name="chassis_bottom_joint" type="fixed">
