Commit message: ok

File: description/lidar.xacro (robot description, xacro)
@@ -4,5 +4,5 @@
         <parent link="chassis"/>
         <child link="laser_frame"/>
-        <origin xyz="0 0 0.5" rpy="0 0 0"/>
+        <origin xyz="0 0 0.5" rpy="0 0 ${pi/2}"/>
     </joint>
     <link name="laser_frame">

File: description/robot_core.xacro (robot description, xacro)
@@ -338,5 +338,5 @@
         <parent link="chassis_bottom"/>
         <child link="laser_frame"/>
-        <origin xyz="0.05 0 0.07" rpy="0 0 0"/>
+        <origin xyz="0.05 0 0.07" rpy="0 0 ${pi/2}"/>
     </joint>
     <link name="laser_frame">
